File: Hardware/GyroX/GyroX_Drone/GyroX_Drone.kicad_sch (KiCad schematic)
At the start: 55 parts, among them J1 USB_C_Receptacle_USB2.0_16P, J2 Conn_01x02, Q1 PMOS, U1 SPX3819M5-L-3-3, U2 CH340K, U3 2N7002DW, U4 TP4056-42-ESOP8, U5 MPU-6050, U6 STM32F405RGTx, U7 BMP390, U8 L86-M33

Commit message: Accelerometer added and power rail filtered
Parts:
- added C4: 100nF, symbol Device:C
- added C5: 10uF, symbol Device:C
- added R19: 10k, symbol Device:R
Connections:
- net +3.3V: now also U8.4 (VCC), U8.5 (V_BCKP), C4.1, C5.1
- net GND: now also C3.2, U7.3 (VSS), U8.12 (GND), U8.3 (GND), C4.2, C5.2
- net BMP_CLK: now reaches U7.2 (SCK)
- net BMP_CSB: now reaches U7.6 (CSB)
- net GPS_RX: now reaches U8.1 (RXD1)
- net at U8.10 (~{RESET}): now also R19.2
- net GPS_TX: now reaches U8.2 (TXD1)
- net MCU_MISO renamed BMP_MISO
- net MCU_MOSI renamed BMP_MOSI
- new net GPS_RST: R19.1
- no-connect marks 3 -> 7
Other:
- note added: "DIGITAL BAROMETRIC PRESSURE SENSOR"
- note added: "GPS SENSOR"
- moved on the sheet: C2, C3, U7, U8
